File: Hardware/Kicad/2025_Animation_Controller.kicad_pcb (KiCad board)
At the start: 4 copper layers, 0 parts

Commit message: Prep for production PCB V1
Parts:
- added C1: 0.1uF, Capacitor_THT:C_Disc_D5.1mm_W3.2mm_P5.00mm, F.Cu at (121.6, 76.0)
- added C10: 0.1uF, Capacitor_THT:C_Disc_D5.1mm_W3.2mm_P5.00mm, F.Cu at (144.8, 111.8)
- added C11: 0.1uF, Capacitor_THT:C_Disc_D5.1mm_W3.2mm_P5.00mm, F.Cu at (144.8, 114.1)
- added C12: 0.1uF, Capacitor_THT:C_Disc_D5.1mm_W3.2mm_P5.00mm, F.Cu at (162.5, 111.8)
- added C13: 0.1uF, Capacitor_THT:C_Disc_D5.1mm_W3.2mm_P5.00mm, F.Cu at (162.5, 114.1)
- added C14: 0.1uF, Capacitor_THT:C_Disc_D5.1mm_W3.2mm_P5.00mm, F.Cu at (103.8, 76.0)
- added C15: 0.1uF, Capacitor_THT:C_Disc_D5.1mm_W3.2mm_P5.00mm, B.Cu at (110.5, 82.7)
- added C16: 10uF-T, Capacitor_THT:CP_Radial_Tantal_D5.5mm_P2.50mm, F.Cu at (165.8, 54.4)
- added C17: 10uF-T, Capacitor_THT:CP_Radial_Tantal_D5.5mm_P2.50mm, F.Cu at (155.8, 65.5)
- added C18: 0.1uF, Capacitor_THT:C_Disc_D5.1mm_W3.2mm_P5.00mm, F.Cu at (160.8, 56.1)
- added C19: 0.1uF, Capacitor_THT:C_Disc_D5.1mm_W3.2mm_P5.00mm, F.Cu at (150.7, 98.1)
- added C2: 0.1uF, Capacitor_THT:C_Disc_D5.1mm_W3.2mm_P5.00mm, F.Cu at (125.5, 76.0)
- added C20: 47uF 35v, Capacitor_THT:CP_Radial_D8.0mm_P3.50mm, F.Cu at (117.8, 50.6)
- added C3: 0.1uF, Capacitor_THT:C_Disc_D5.1mm_W3.2mm_P5.00mm, F.Cu at (145.9, 76.1)
- added C4: 0.1uF, Capacitor_THT:C_Disc_D5.1mm_W3.2mm_P5.00mm, F.Cu at (169.8, 96.5)
- added C5: 0.1uF, Capacitor_THT:C_Disc_D5.1mm_W3.2mm_P5.00mm, F.Cu at (164.4, 58.4)
- added C6: 0.1uF, Capacitor_THT:C_Disc_D5.1mm_W3.2mm_P5.00mm, F.Cu at (109.3, 111.8)
- added C7: 0.1uF, Capacitor_THT:C_Disc_D5.1mm_W3.2mm_P5.00mm, F.Cu at (109.3, 114.1)
- added C8: 0.1uF, Capacitor_THT:C_Disc_D5.1mm_W3.2mm_P5.00mm, F.Cu at (127.0, 111.8)
- added C9: 0.1uF, Capacitor_THT:C_Disc_D5.1mm_W3.2mm_P5.00mm, F.Cu at (127.0, 114.1)
- added D2: 5KP18A, Diode_THT:D_P600_R-6_P12.70mm_Horizontal, F.Cu at (111.5, 51.4)
- added D3: Ideal Diode, 1_Joe_Footprints:Ideal_Diode_AGM403A, F.Cu at (113.8, 63.0)
- added F1: Polyfuse 5A, Fuse:Fuse_Littelfuse_395Series, F.Cu at (115.6, 55.5)
- added H1: MountingHole, MountingHole:MountingHole_3.2mm_M3, F.Cu at (96.9, 41.9)
- added H2: MountingHole, MountingHole:MountingHole_3.2mm_M3, F.Cu at (209.9, 41.9)
- added H3: MountingHole, MountingHole:MountingHole_3.2mm_M3, F.Cu at (209.9, 118.9)
- added H4: MountingHole, MountingHole:MountingHole_3.2mm_M3, F.Cu at (96.9, 118.9)
- added J1: I2C2 Bus, Connector_JST:JST_XH_B4B-XH-A_1x04_P2.50mm_Vertical, F.Cu at (155.8, 100.2)
- added J10: Conn_01x02, Connector_JST:JST_XH_B2B-XH-A_1x02_P2.50mm_Vertical, F.Cu at (177.8, 105.5)
- added J11: Conn_01x02, Connector_JST:JST_XH_B2B-XH-A_1x02_P2.50mm_Vertical, F.Cu at (177.4, 116.8)
- added J12: Conn_01x02, Connector_JST:JST_XH_B2B-XH-A_1x02_P2.50mm_Vertical, F.Cu at (186.9, 105.5)
- added J13: Conn_01x02, Connector_JST:JST_XH_B2B-XH-A_1x02_P2.50mm_Vertical, F.Cu at (186.1, 116.8)
- added J14: Conn_01x02, Connector_JST:JST_XH_B2B-XH-A_1x02_P2.50mm_Vertical, F.Cu at (196.0, 105.5)
- added J15: Conn_01x02, Connector_JST:JST_XH_B2B-XH-A_1x02_P2.50mm_Vertical, F.Cu at (194.8, 116.8)
- added J16: Conn_01x02, Connector_JST:JST_XH_B2B-XH-A_1x02_P2.50mm_Vertical, F.Cu at (205.0, 105.5)
- added J17: Conn_01x02, Connector_JST:JST_XH_B2B-XH-A_1x02_P2.50mm_Vertical, F.Cu at (203.5, 116.8)
- added J18: Enc, Connector_JST:JST_XH_B4B-XH-A_1x04_P2.50mm_Vertical, F.Cu at (116.6, 74.2)
- added J19: Speed Pot, JST-XH, Connector_JST:JST_XH_B3B-XH-A_1x03_P2.50mm_Vertical, F.Cu at (131.5, 69.1)
- added J2: Conn_01x02, Connector_JST:JST_XH_B2B-XH-A_1x02_P2.50mm_Vertical, F.Cu at (169.5, 45.4)
- added J20: Speed Pot, JST-XH, Connector_JST:JST_XH_B3B-XH-A_1x03_P2.50mm_Vertical, F.Cu at (139.8, 69.1)
- added J21: LCD Display, Connector_JST:JST_XH_B7B-XH-A_1x07_P2.50mm_Vertical, F.Cu at (166.4, 73.7)
- added J22: Serial 1, Connector_JST:JST_XH_B4B-XH-A_1x04_P2.50mm_Vertical, F.Cu at (104.4, 109.0)
- added J23: Serial 2, Connector_JST:JST_XH_B4B-XH-A_1x04_P2.50mm_Vertical, F.Cu at (115.2, 109.0)
- added J24: Serial 3, Connector_JST:JST_XH_B4B-XH-A_1x04_P2.50mm_Vertical, F.Cu at (122.1, 109.0)
- added J25: Serial 4, Connector_JST:JST_XH_B4B-XH-A_1x04_P2.50mm_Vertical, F.Cu at (132.9, 109.0)
- added J26: Serial 5, Connector_JST:JST_XH_B4B-XH-A_1x04_P2.50mm_Vertical, F.Cu at (139.9, 109.0)
- added J27: Serial 6, Connector_JST:JST_XH_B4B-XH-A_1x04_P2.50mm_Vertical, F.Cu at (150.7, 109.0)
- added J28: Serial 7, Connector_JST:JST_XH_B4B-XH-A_1x04_P2.50mm_Vertical, F.Cu at (157.6, 109.0)
- added J29: Serial 8, Connector_JST:JST_XH_B4B-XH-A_1x04_P2.50mm_Vertical, F.Cu at (168.4, 109.0)
- added J3: Conn_01x02, Connector_JST:JST_XH_B2B-XH-A_1x02_P2.50mm_Vertical, F.Cu at (177.8, 45.4)
- added J30: 12V in, Connector_JST:JST_XH_B2B-XH-AM_1x02_P2.50mm_Vertical, F.Cu at (102.2, 62.0)
- added J31: Spares A, Connector_JST:JST_XH_B8B-XH-A_1x08_P2.50mm_Vertical, F.Cu at (101.7, 100.6)
- added J32: Spares B, Connector_JST:JST_XH_B8B-XH-A_1x08_P2.50mm_Vertical, F.Cu at (126.8, 100.5)
- added J4: Conn_01x02, Connector_JST:JST_XH_B2B-XH-A_1x02_P2.50mm_Vertical, F.Cu at (186.1, 45.4)
- added J5: Conn_01x02, Connector_JST:JST_XH_B2B-XH-A_1x02_P2.50mm_Vertical, F.Cu at (194.4, 45.4)
- added J6: Conn_01x02, Connector_JST:JST_XH_B2B-XH-A_1x02_P2.50mm_Vertical, F.Cu at (202.5, 45.5)
- added J7: Conn_01x02, Connector_JST:JST_XH_B2B-XH-A_1x02_P2.50mm_Vertical, F.Cu at (205.1, 69.3)
- added J8: Conn_01x02, Connector_JST:JST_XH_B2B-XH-A_1x02_P2.50mm_Vertical, F.Cu at (205.1, 61.1)
- added J9: Conn_01x02, Connector_JST:JST_XH_B2B-XH-A_1x02_P2.50mm_Vertical, F.Cu at (205.0, 52.8)
- added JP1: Display Pwr, Connector_PinHeader_2.54mm:PinHeader_1x03_P2.54mm_Vertical, F.Cu at (165.3, 63.3)
- added R1: 2.2K, Resistor_THT:R_Axial_DIN0207_L6.3mm_D2.5mm_P10.16mm_Horizontal, B.Cu at (166.6, 91.8)
- added R2: 2.2K, Resistor_THT:R_Axial_DIN0207_L6.3mm_D2.5mm_P10.16mm_Horizontal, B.Cu at (169.7, 81.6)
- added R3: 10k, Resistor_THT:R_Axial_DIN0207_L6.3mm_D2.5mm_P10.16mm_Horizontal, B.Cu at (116.0, 80.9)
- added R4: 10k, Resistor_THT:R_Axial_DIN0207_L6.3mm_D2.5mm_P10.16mm_Horizontal, B.Cu at (119.2, 80.9)
- added TP1: GND, TestPoint:TestPoint_Plated_Hole_D2.0mm, F.Cu at (107.7, 43.2)
- added TP2: 12V, TestPoint:TestPoint_Plated_Hole_D2.0mm, F.Cu at (113.4, 43.3)
- added TP3: 5V, TestPoint:TestPoint_Plated_Hole_D2.0mm, F.Cu at (148.1, 67.8)
- added TP4: 3.3AUX, TestPoint:TestPoint_Plated_Hole_D2.0mm, F.Cu at (174.7, 56.4)
- added U1: ULN2803, 1_Joe_Footprints:ULN2803_Breakout_Board, F.Cu at (189.6, 61.6)
- added U2: Teensy4.1, teensy.pretty-master:Teensy41, F.Cu at (132.4, 86.2)
- added U3: DFR1015, 1_Joe_Footprints:DCDC_Converter_DFR1015, F.Cu at (138.0, 53.9)
- added U4: LM1117T-3.3, Package_TO_SOT_THT:TO-220-3_Vertical, F.Cu at (155.3, 53.6)
- added U5: I/O Expander, 1_Joe_Footprints:SX1509_Breakout_Board, F.Cu at (169.9, 88.5)
Routing:
- net /SX1509_INT: track 0.00 -> 67.7 mm
- net /I2C_SCL: track 0.00 -> 55.7 mm
- net /I2C_SDA: track 0.00 -> 53.3 mm
- net /REMOTE_ACT_5_RX: track 0.00 -> 48.8 mm, vias 0 -> 2
- net /REMOTE_ACT_4_TX: track 0.00 -> 48.7 mm, vias 0 -> 1
- net /REMOTE_ACT_8_TX: track 0.00 -> 48.3 mm, vias 0 -> 2
- net /SPARE_23: track 0.00 -> 47.5 mm, vias 0 -> 1
- net /REMOTE_ACT_4_RX: track 0.00 -> 47.2 mm, vias 0 -> 1
- net /REMOTE_ACT_5_TX: track 0.00 -> 45.2 mm, vias 0 -> 2
- net /REMOTE_ACT_8_RX: track 0.00 -> 44.2 mm, vias 0 -> 1
- net /REMOTE_ACT_3_RX: track 0.00 -> 43.6 mm
- net /SPARE_33: track 0.00 -> 40.3 mm
- net /REMOTE_ACT_3_TX: track 0.00 -> 40.3 mm
- net /SPARE_27: track 0.00 -> 39.9 mm, vias 0 -> 3
- net /SPARE_26: track 0.00 -> 37.5 mm, vias 0 -> 2
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- added copper zone on In2.Cu, net +12V
- added copper zone on In2.Cu, net +5V
- added copper zone on In2.Cu, net /Display_Power
- added copper zone on In2.Cu, net 3V3_AUX
- added copper zone on In2.Cu, net 3V3_MCU
- added copper zone on In1.Cu, net GND
Other:
- board outline added: 120 x 84 mm
- board text added: "+ GND"
- board text added: "12V"
- board text added: "12V In"
- board text added: "3V3"
- board text added: "3V3-AUX"
- board text added: "3V3_MCU"
- board text added: "5V"
- board text added: "5v-|-3v3"
- board text added: "Accel Pot"
- board text added: "BTN 1"
- board text added: "BTN 2"
- board text added: "BTN 3"
- board text added: "BTN 4"
- board text added: "BTN 5"
- board text added: "BTN 6"
- board text added: "BTN 7"
- board text added: "BTN 8"
- board text added: "Display SPI"
- board text added: "ENC"
- board text added: "G"
- board text added: "GND"
- board text added: "I2C2 Bus"
- board text added: "LED 1"
- board text added: "LED 2"
- board text added: "LED 3"
- board text added: "LED 4"
- board text added: "LED 5"
- board text added: "LED 6"
- board text added: "LED 7"
- board text added: "LED 8"
- board text added: "RX"
- board text added: "Robotic Animation Controller Ver 1 ©2025 JM Designs"
- board text added: "SER-1"
- board text added: "SER-2"
- board text added: "SER-3"
- board text added: "SER-4"
- board text added: "SER-5"
- board text added: "SER-6"
- board text added: "SER-7"
- board text added: "SER-8"
- board text added: "SPARES-A"
- board text added: "SPARES-B"
- board text added: "Speed Pot"
- board text added: "TX"
- board text added: "USB"
