File: Hardware/Kicad/2025_Animation_Controller.kicad_sch (KiCad schematic)
At the start: 61 parts, among them J1 I2C2 Bus, J10 Conn_01x02, J11 Conn_01x02, J12 Conn_01x02, J13 Conn_01x02, J14 Conn_01x02, J15 Conn_01x02, J16 Conn_01x02, J17 Conn_01x02, J18 Jog Encoder, JST XH, J19 Speed Pot, JST-XH, J2 Conn_01x02, J20 Speed Pot, JST-XH, J21 Display, JST-XH, J22 Serial 1, J23 Serial 2, J24 Serial 3, J25 Serial 4, J26 Serial 5, J27 Serial 6, J28 Serial 7, J29 Serial 8, J3 Conn_01x02, J30 Power Term Block, J31 Spares A, J32 Spares B, J4 Conn_01x02, J5 Conn_01x02, J6 Conn_01x02, J7 Conn_01x02, J8 Conn_01x02, J9 Conn_01x02, U1 SX1509, U2 Teensy4.1, U3 ULN2803A

Commit message: Prep for production PCB V1
Parts:
- removed D1: SMAJ13A, Diode_SMD:D_SMA, symbol Diode:SMAJ13A
- removed U1: SX1509, PCM_SparkFun-Semiconductor-Standard:QFN-28-1EP_4x4mm_P0.4mm_EP2.6x2.6mm, symbol PCM_SparkFun-IC-Special-Function:SX1509
- removed U3: ULN2803A, symbol Transistor_Array:ULN2803A
- removed U4: ~, symbol Joe_Mohos_Symbols:DCDC_Converter_LM2596_3A
- added C16, C17: 10uF-T, Capacitor_THT:CP_Radial_Tantal_D5.5mm_P2.50mm, symbol Device:C_Polarized_Small
- added C18, C19: 0.1uF, Capacitor_THT:C_Disc_D5.1mm_W3.2mm_P5.00mm, symbol Device:C_Small
- added C20: 47uF 35v, Capacitor_THT:CP_Radial_D8.0mm_P3.50mm, symbol Device:C_Polarized_Small
- added D3: Ideal Diode, 1_Joe_Footprints:Ideal_Diode_AGM403A, symbol Joe_Mohos_Symbols:Ideal_Diode_Board
- added R3, R4: 10k, Resistor_THT:R_Axial_DIN0207_L6.3mm_D2.5mm_P10.16mm_Horizontal, symbol Device:R
- added TP1: GND, TestPoint:TestPoint_Plated_Hole_D2.0mm, symbol Connector:TestPoint
- added TP2: 12V, TestPoint:TestPoint_Plated_Hole_D2.0mm, symbol Connector:TestPoint
- added TP3: 5V, TestPoint:TestPoint_Plated_Hole_D2.0mm, symbol Connector:TestPoint
- added TP4: 3.3AUX, TestPoint:TestPoint_Plated_Hole_D2.0mm, symbol Connector:TestPoint
- added U1: ULN2803, 1_Joe_Footprints:ULN2803_Breakout_Board, symbol Joe_Mohos_Symbols:ULN2803_Breakout_Board
- added U3: DFR1015, 1_Joe_Footprints:DCDC_Converter_DFR1015, symbol Joe_Mohos_Symbols:DCDC_Converter_DFR1015
- added U4: LM1117T-3.3, Package_TO_SOT_THT:TO-220-3_Vertical, symbol Regulator_Linear:LM1117T-3.3
- added U5: I/O Expander, 1_Joe_Footprints:SX1509_Breakout_Board, symbol Joe_Mohos_Symbols:SX1509_Breakout_Board
- C1, C10, C11, C12, C13, C14, C15, C2, C3, C4, C5, C6, C7, C8, C9: footprint (none) -> Capacitor_THT:C_Disc_D5.1mm_W3.2mm_P5.00mm
- D2: value Ideal Diode -> 5KP18A; footprint (none) -> Diode_THT:D_P600_R-6_P12.70mm_Horizontal
- F1: footprint (none) -> Fuse:Fuse_Littelfuse_395Series
- J1, J22, J23, J24, J25, J26, J27, J28, J29: footprint (none) -> Connector_JST:JST_XH_B4B-XH-A_1x04_P2.50mm_Vertical
- J10, J11, J12, J13, J14, J15, J16, J17, J2, J3, J4, J5, J6, J7, J8, J9: footprint (none) -> Connector_JST:JST_XH_B2B-XH-A_1x02_P2.50mm_Vertical
- J18: value Jog Encoder, JST XH -> Enc; footprint (none) -> Connector_JST:JST_XH_B4B-XH-A_1x04_P2.50mm_Vertical
- J19, J20: footprint (none) -> Connector_JST:JST_XH_B3B-XH-A_1x03_P2.50mm_Vertical
- J21: value Display, JST-XH -> LCD Display; footprint (none) -> Connector_JST:JST_XH_B7B-XH-A_1x07_P2.50mm_Vertical
- J30: value Power Term Block -> 12V in; footprint (none) -> Connector_JST:JST_XH_B2B-XH-AM_1x02_P2.50mm_Vertical; symbol Connector:Screw_Terminal_01x02 -> Connector_Generic:Conn_01x02
- J31, J32: footprint (none) -> Connector_JST:JST_XH_B8B-XH-A_1x08_P2.50mm_Vertical
- JP1: footprint (none) -> Connector_PinHeader_2.54mm:PinHeader_1x03_P2.54mm_Vertical
- U2: footprint (none) -> teensy.pretty-master:Teensy41; symbol teensy:Teensy4.1 -> Joe_Mohos_Symbols:Teensy4.1
Connections:
- net +12V: now also D2.1 (K), C20.1, TP2.1, U1.10 (COM), U3.3 (Vin+), U3.4 (Vin+)
- net +5V: now also C17.1, TP3.1, U3.5 (Vout+), U3.6 (Vout+), U4.3 (VI)
- net BUTTON_1: now also U5.14 (P0)
- net BUTTON_2: now also U5.15 (P1)
- net BUTTON_3: now also U5.16 (P2)
- net BUTTON_4: now also U5.17 (P3)
- net BUTTON_5: now also U5.19 (P4)
- net BUTTON_6: now also U5.20 (P5)
- net BUTTON_7: now also U5.21 (P6)
- net BUTTON_8: now also U5.22 (P7)
- net ENCODER_A: now also R4.2
- net ENCODER_B: now also R3.2
- net GND: now also D2.2 (A), C16.2, C17.2, C18.2, C19.1, C20.2, TP1.1, U1.9 (GND), U3.1 (Vin-), U3.2 (Vin-), U3.7 (Vout-), U3.8 (Vout-), U4.1 (GND), U5.13 (GND), U5.3 (GND), U5.32 (GND), U5.33 (GND), U5.34 (P15_COM), U5.35 (P14_COM), U5.36 (P13_COM), U5.37 (P12_COM), U5.38 (VC2_COM), U5.39 (P11_COM), U5.40 (P10_COM), U5.41 (P9_COM), U5.42 (P8_COM), U5.43 (P7_COM), U5.44 (P6_COM), U5.45 (P5_COM), U5.46 (P4_COM), U5.47 (VC1_COM), U5.48 (P3_COM), U5.49 (P2_COM), U5.50 (P1_COM), U5.51 (P0_COM), U5.52 (GND), U5.9 (GND)
- net I2C_SCL: now also U5.6 (~{SCL})
- net I2C_SDA: now also U5.5 (~{SDA})
- net LED_1: now also U1.1 (IN1), U5.31 (P15)
- net LED_1_12V: now also U1.18 (OUT1)
- net LED_2: now also U1.2 (IN2), U5.30 (P14)
- net LED_2_12V: now also U1.17 (OUT2)
- net LED_3: now also U1.3 (IN3), U5.29 (P13)
- net LED_3_12V: now also U1.16 (OUT3)
- net LED_4: now also U1.4 (IN4), U5.28 (P12)
- net LED_4_12V: now also U1.15 (OUT4)
- net LED_5: now also U1.5 (IN5), U5.26 (P11)
- net LED_5_12V: now also U1.14 (OUT5)
- net LED_6: now also U1.6 (IN6), U5.25 (P10)
- net LED_6_12V: now also U1.13 (OUT6)
- net LED_7: now also U1.7 (IN7), U5.24 (P9)
- net LED_7_12V: now also U1.12 (OUT7)
- net LED_8: now also U1.8 (IN8), U5.23 (P8)
- net LED_8_12V: now also U1.11 (OUT8)
- net SX1509_INT: now also U5.1 (~{INT})
- net at J30.2 (Pin_2): now also D3.1, D3.2; no longer D2.2 (A)
- net at F1.1: now also D3.3, D3.4; no longer D2.1 (K)
- net +3.3V renamed 3V3_AUX
- net 3V3_AUX: now also C16.1, C18.1, C19.2, TP4.1, U4.2 (VO), U5.4 (3V3); no longer C1.1, C15.1, C2.1, C3.1, J18.2 (Pin_2), J19.3 (Pin_3), J20.3 (Pin_3), U2.15 (3V3), U2.46 (3V3)
- net SPI_MISO: no longer names the net of U2.14 (12_MISO_MQSL)
- new net 3V3_MCU: C1.1, C15.1, C2.1, C3.1, J18.2 (Pin_2), J19.3 (Pin_3), J20.3 (Pin_3), R3.1, R4.1, U2.15 (3V3), U2.46 (3V3)
- no-connect marks 1 -> 10
Other:
- note added: "Buttons and LED Connectors"
- note added: "I/O Expander and Driver"
- note added: "TVS, 18V 5000W"
- note added: "Test Points"
- note removed: "Buttons and LEDs"
- moved on the sheet: C1, C14, C15, C2, C3, C4, F1, J1, J10, J11, J12, J13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

Commit message: First working edit revision.
Other:
- title: (none) -> Robotic Animation Controller
Changed lines of the file:
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@@
 	(generator_version "9.0")
 	(paper "A4")
+	(title_block
+		(title "Robotic Animation Controller")
+		(date "2026-01-09")
+		(rev "V1")
+	)
 	(rectangle
 		(start 116.84 132.715)
